Commit message: added a decimation that makes walking more stable

File: genesis/assets/urdf/aliengo/urdf/aliengo.urdf (robot description, URDF)
Before this commit: robot aliengo, 18 links, 17 joints
Joints:
- joint FL_calf_joint: limit lower=-2.775073510670984 upper=-0.6457718232379019 effort=44.4 velocity=15.89 -> lower=-2.775 upper=-0.611 effort=44.4 velocity=15.89
- joint FR_calf_joint: limit lower=-2.775073510670984 upper=-0.6457718232379019 effort=44.4 velocity=15.89 -> lower=-2.775 upper=-0.611 effort=44.4 velocity=15.89
- joint RL_calf_joint: limit lower=-2.775073510670984 upper=-0.6457718232379019 effort=44.4 velocity=15.89 -> lower=-2.775 upper=-0.611 effort=44.4 velocity=15.89
- joint RR_calf_joint: limit lower=-2.775073510670984 upper=-0.6457718232379019 effort=44.4 velocity=15.89 -> lower=-2.775 upper=-0.611 effort=44.4 velocity=15.89

File: genesis/assets/urdf/go1/urdf/go1.urdf (robot description, URDF)
Before this commit: robot go1, 19 links, 18 joints
Joints:
- joint FL_calf_joint: limit lower=-2.818 upper=-0.888 effort=35.55 velocity=20.06 -> lower=-2.721 upper=-0.837 effort=35.55 velocity=20.06
- joint FL_hip_joint: limit lower=-0.863 upper=0.863 effort=23.7 velocity=30.1 -> lower=-1.047 upper=1.047 effort=23.7 velocity=30.1
- joint FL_thigh_joint: limit lower=-0.686 upper=4.501 effort=23.7 velocity=30.1 -> lower=-0.663 upper=2.966 effort=23.7 velocity=30.1
- joint FR_calf_joint: limit lower=-2.818 upper=-0.888 effort=35.55 velocity=20.06 -> lower=-2.721 upper=-0.837 effort=35.55 velocity=20.06
- joint FR_hip_joint: limit lower=-0.863 upper=0.863 effort=23.7 velocity=30.1 -> lower=-1.047 upper=1.047 effort=23.7 velocity=30.1
- joint FR_thigh_joint: limit lower=-0.686 upper=4.501 effort=23.7 velocity=30.1 -> lower=-0.663 upper=2.966 effort=23.7 velocity=30.1
- joint RL_calf_joint: limit lower=-2.818 upper=-0.888 effort=35.55 velocity=20.06 -> lower=-2.721 upper=-0.837 effort=35.55 velocity=20.06
- joint RL_hip_joint: limit lower=-0.863 upper=0.863 effort=23.7 velocity=30.1 -> lower=-1.047 upper=1.047 effort=23.7 velocity=30.1
- joint RL_thigh_joint: limit lower=-0.686 upper=4.501 effort=23.7 velocity=30.1 -> lower=-0.663 upper=2.966 effort=23.7 velocity=30.1
- joint RR_calf_joint: limit lower=-2.818 upper=-0.888 effort=35.55 velocity=20.06 -> lower=-2.721 upper=-0.837 effort=35.55 velocity=20.06
- joint RR_hip_joint: limit lower=-0.863 upper=0.863 effort=23.7 velocity=30.1 -> lower=-1.047 upper=1.047 effort=23.7 velocity=30.1
- joint RR_thigh_joint: limit lower=-0.686 upper=4.501 effort=23.7 velocity=30.1 -> lower=-0.663 upper=2.966 effort=23.7 velocity=30.1
