Commit message: Ignore CI script 'setup_env.sh' return code.

File: genesis/assets/urdf/3763/mobility.urdf (robot description, URDF)
Before this commit: robot partnet_6b8b2cb01c376064c8724d5673a063a6, 4 links, 3 joints
Joints:
- joint joint_2: limit lower=-0.1080000000000001 upper=-z0.008000000000000007 -> lower=-0.1080000000000001 upper=-0.008000000000000007
