Commit message: Fix naming convention inconsistencies.

File: genesis/assets/urdf/shadow_hand/shadow_hand.urdf (robot description, URDF)
Before this commit: robot shadow_hand, 25 links, 24 joints
Joints:
- removed joint index_finger_join2
- added joint index_finger_joint2: type revolute, parent index_finger_knuckle, child index_finger_proximal, axis 1 0 0, limit lower=0 upper=1.57079632679 effort=4.0 velocity=2.0
