Commit message: Ipc coupling 0126 (#3)
* Optimize IPC coupling with Taichi fields and kernel improvements

- Replace ndarray parameters with ti.template() in all kernels for better performance
- Add Taichi fields to store link states (pos/quat) and qpos across coupling strategies
- Add ArticulationData class for external_articulation coupling
- Add kernels: _store_link_states, _store_qpos, _copy_stored_qpos_to_articulation
- Store qpos once in _store_genesis_rigid_states, reuse across all couplings
- Add prev_link_transforms dict to ArticulationData for reference tracking

* Remove temporary numpy arrays in external_articulation coupling

- Remove temporary delta_theta_tilde numpy array, write directly to IPC view
- Remove temporary delta_theta_ipc numpy array, read directly from IPC view
- Remove large qpos_new_batch array, extract qpos per entity on-demand
- Add _update_ref_dof_prev_kernel for parallelized ref_dof_prev update
- Replace Python loops with direct Taichi field access where possible

Performance improvements:
- Eliminated 3 large temporary numpy array allocations per coupling step
- Reduced memory copying overhead
- Better memory locality with direct field-to-view transfers

* Add separate kernels for ti.field and ti.ndarray to support both use_ndarray modes

* fix

* bug fix

* multiple tests

* add options

* testing

* fix api mismatching problem, still problem in rigid coupling in ipc_cloth.py

* add a uipc setup test

* update example

* update semi implicit option

* add a minimal example of loading panda_non_overlap

* update joint axis

* fix joint

* bug fix for get_all_pos

* fix following problem

* update options

* new framework for coupling. supports multi coupling strategy.

* bug fix

* workaround for demo

* use forward kinematic to update Genesis robot

* refactor(ipc_coupler): reorganize into package structure with data.py and utils.py

- Split ipc_coupler.py into a package with:
  - coupler.py: Main IPCCoupler class with Taichi kernels
  - data.py: Taichi data-oriented classes (IPCTransformData, IPCCouplingData, ArticulationData)
  - utils.py: Utility functions extracted from coupler
  - __init__.py: Package exports

- Add class constants for buffer sizes (MAX_CONTACTS, MAX_LINKS, etc.)
- Optimize batch processing for force/torque application

* perf(ipc_coupler): optimize numpy array operations

* cleanup

* cleanup

---------

Co-authored-by: TempContainer <wangzhny@gmail.com>
Co-authored-by: Zhaofeng Luo <zhaofen2@andrew.cmu.edu>

File: genesis/assets/urdf/simple/three_cube_chain.urdf (robot description, URDF)
Before this commit: robot three_cube_chain, 3 links, 2 joints
Joints:
- joint joint2: axis 0 0 1 -> 0 1 0
