Commit message: fix(urdf): add missing inertial blocks to panda_slider_mobile base links
The planar-base intermediate links (basex, basey, basez, base) in
panda_slider_mobile.urdf were self-closing elements with no inertial
blocks. Genesis legacy parser assigns gs.EPS (~1e-15) mass to these
movable links, causing numerical instability when the Franka arm
accelerates while gripping a payload.

Added inertial blocks with reasonable default mass values:
- basex/basey/basez: 1.0 kg each (intermediate slider/prismatic links)
- base: 20.0 kg (base plate supporting the robot arm)

Reproduced on ROCm/HIP 7.2, AMD Radeon PRO W7900 (gfx1100), Genesis 1.3.0.

Closes #3185

File: genesis/assets/urdf/panda_bullet/panda_slider_mobile.urdf (robot description, URDF)
Before this commit: robot panda, 17 links, 16 joints
Links:
- link base: mass None -> 20.0
- link basex: mass None -> 1.0
- link basey: mass None -> 1.0
- link basez: mass None -> 1.0
